File: trunk/KiCAD_ExpansionBoard/External_connectors.sch (KiCad schematic (older format))
At the start: 0 parts

Commit message: Creation of project (sheets) structure and add some library schematic component (transceiver.lib, headers, etc.)
Parts:
- added P?: UART1, symbol CONN_3X2
- added P?: UART2, symbol CONN_3X2
Changed lines of the file:
@@
 EESchema Schematic File Version 2
+LIBS:boosterpack
 LIBS:power
 LIBS:device
@@
 LIBS:contrib
 LIBS:valves
+LIBS:transceiver
 LIBS:TM4C123G_CommExpBoard-cache
 EELAYER 27 0
@@
 Date "9 jun 2014"
 Rev "0.1"
-Comp "Luca Buccolini, student @ Università Politecnica delle Marche"
+Comp "Luca Buccolini, Student @ Università Politecnica delle Marche"
 Comment1 "Expansion Board for the Texas Instruments TM4C123G Launchpad "
 Comment2 ""
@@
 Comment4 ""
 $EndDescr
+$Comp
+L CONN_3X2 P?
+U 1 1 5395F25D
+P 4000 3600
+F 0 "P?" H 4000 3850 50  0000 C CNN
+F 1 "UART1" V 4000 3650 40  0000 C CNN
+F 2 "" H 4000 3600 60  0000 C CNN
+F 3 "http://www.farnell.com/datasheets/1697530.pdf" H 4000 3600 60  0001 C CNN
+F 4 "Farnell" H 4000 3600 60  0001 C CNN "Supplier 1"
+F 5 "1593440" H 4000 3600 60  0001 C CNN "Supplier 1 P/N"
+F 6 "Multicomp" H 4000 3600 60  0001 C CNN "Producer"
+F 7 "2213S-06G" H 4000 3600 60  0001 C CNN "Producer P/N"
+	1    4000 3600
+	1    0    0    -1
+$EndComp
+$Comp
+L CONN_3X2 P?
+U 1 1 5395F8F1
+P 5200 3600
+F 0 "P?" H 5200 3850 50  0000 C CNN
+F 1 "UART2" V 5200 3650 40  0000 C CNN
+F 2 "" H 5200 3600 60  0000 C CNN
+F 3 "http://www.farnell.com/datasheets/1697530.pdf" H 5200 3600 60  0001 C CNN
+F 4 "Farnell" H 5200 3600 60  0001 C CNN "Supplier 1"
+F 5 "1593440" H 5200 3600 60  0001 C CNN "Supplier 1 P/N"
+F 6 "Multicomp" H 5200 3600 60  0001 C CNN "Producer"
+F 7 "2213S-06G" H 5200 3600 60  0001 C CNN "Producer P/N"
+	1    5200 3600
+	1    0    0    -1
+$EndComp
 $EndSCHEMATC

Commit message: Circuit board schematic complete! TODO: Update schematic according new received specifics: "note-expansionboard_20140623.txt"
Parts:
- removed P?: UART1, symbol CONN_3X2
- removed P?: UART2, symbol CONN_3X2
Changed lines of the file:
@@
 EESchema Schematic File Version 2
+LIBS:cdsot23-sm712
+LIBS:TPS62160
 LIBS:boosterpack
 LIBS:power
@@
 Sheet 2 4
 Title "TM4C123G Communication Expansion Board"
-Date "9 jun 2014"
+Date "10 jun 2014"
 Rev "0.1"
 Comp "Luca Buccolini, Student @ Università Politecnica delle Marche"
@@
 Comment4 ""
 $EndDescr
-$Comp
-L CONN_3X2 P?
-U 1 1 5395F25D
-P 4000 3600
-F 0 "P?" H 4000 3850 50  0000 C CNN
-F 1 "UART1" V 4000 3650 40  0000 C CNN
-F 2 "" H 4000 3600 60  0000 C CNN
-F 3 "http://www.farnell.com/datasheets/1697530.pdf" H 4000 3600 60  0001 C CNN
-F 4 "Farnell" H 4000 3600 60  0001 C CNN "Supplier 1"
-F 5 "1593440" H 4000 3600 60  0001 C CNN "Supplier 1 P/N"
-F 6 "Multicomp" H 4000 3600 60  0001 C CNN "Producer"
-F 7 "2213S-06G" H 4000 3600 60  0001 C CNN "Producer P/N"
-	1    4000 3600
-	1    0    0    -1
-$EndComp
-$Comp
-L CONN_3X2 P?
-U 1 1 5395F8F1
-P 5200 3600
-F 0 "P?" H 5200 3850 50  0000 C CNN
-F 1 "UART2" V 5200 3650 40  0000 C CNN
-F 2 "" H 5200 3600 60  0000 C CNN
-F 3 "http://www.farnell.com/datasheets/1697530.pdf" H 5200 3600 60  0001 C CNN
-F 4 "Farnell" H 5200 3600 60  0001 C CNN "Supplier 1"
-F 5 "1593440" H 5200 3600 60  0001 C CNN "Supplier 1 P/N"
-F 6 "Multicomp" H 5200 3600 60  0001 C CNN "Producer"
-F 7 "2213S-06G" H 5200 3600 60  0001 C CNN "Producer P/N"
-	1    5200 3600
-	1    0    0    -1
-$EndComp
 $EndSCHEMATC
