File: trunk/KiCAD_ExpansionBoard/Expansion_board.sch (KiCad schematic (older format))
At the start: 35 parts, among them P1 ANT_GND, P5 ANT_C, Q1 NTR4101P, Q3 PDTC124XT, SW1 SLIDE_SWITCH_SPDT, SW2 SLIDE_SWITCH_4PDT, U1 SN65HVD234, U2 TPS62160, U3 SN65HVD11, U4 RFM23B

Commit message: - sostituiti i pad smd dell'antenna con due pad through hole; - ridotto il numero di vias sottostanti il modulo radio RFM23B e spostati i rimanenti in maniera da evitare la sovrapposizione con i vias del modulo; - eliminate le zone di rame fra i pin dei componenti più piccoli come i resistori e condensatori 0805; - eliminati i vias vicino ai connettori "pin-header" e connesse le piste ai connettori direttamente dal lato bottom; - sostituiti i resistori di pull-up e pull-down della rete di fail-safe-bias con dei resistori di valore doppio circa (560->1k2);
Aggiunta la cartella "PCB_fabrication" che contiene:
- il file excel (BOM);
- i file per le forature;
- i file Gerber;
- alcuni file .txt che descrivono il contenuto delle rispettive cartelle.
Parts:
- R13, R15: value 560 -> 1k2; Descriprion RESISTORE, 560R, 0.125W, 1%, 0805, SMD -> WELWYN WCR0805-1K2FI RESISTORE, 0805 1K2; Producer VISHAY DRALORIC -> WELWYN; Producer P/N CRCW0805560RFKEA -> WCR0805-1K2FI; Supplier 1 P/N 1469945 -> 1100315
